Commit message: fix bug and add barrett move (grasp) func

File: data_robot/urdfs/barrett/bh282.urdf (robot description, URDF)
Before this commit: robot bhand_, 12 links, 11 joints
Links:
- link base_link: mass None -> 0.8
- link bh_base_link: mass 1.0 -> 0.8
- link hand_base_link: mass None -> 0.8

Commit message: fix minor bug

File: data_robot/urdfs/barrett/bh282.urdf (robot description, URDF)
Before this commit: robot bhand_, 12 links, 11 joints
Links:
- link bh_finger_11_link: mass 0.1 -> 0.8
- link bh_finger_12_link: mass 0.1 -> 0.8
- link bh_finger_13_link: mass 0.1 -> 0.8
- link bh_finger_21_link: mass 0.1 -> 0.8
- link bh_finger_22_link: mass 0.1 -> 0.8
- link bh_finger_23_link: mass 0.1 -> 0.8
- link bh_finger_31_link: mass 0.1 -> 0.8
- link bh_finger_32_link: mass 0.1 -> 0.8
- link bh_finger_33_link: mass 0.1 -> 0.8

Commit message: simplify mesh and tune bullet for stable data col

File: data_robot/urdfs/barrett/bh282.urdf (robot description, URDF)
Before this commit: robot bhand_, 12 links, 11 joints
Joints:
- joint bh_j11_joint: limit lower=0 upper=3.1416 effort=30.0 velocity=2.0 -> lower=0 upper=3.1416 effort=30.0 velocity=0.2; type revolute -> fixed
- joint bh_j12_joint: limit lower=0.0 upper=2.44 effort=30.0 velocity=2.0 -> lower=0.0 upper=2.44 effort=30.0 velocity=0.2
- joint bh_j13_joint: limit lower=0.0 upper=0.84 effort=30.0 velocity=2.0 -> lower=0.0 upper=0.84 effort=30.0 velocity=0.2
- joint bh_j21_joint: limit lower=0 upper=3.1416 effort=30.0 velocity=2.0 -> lower=0 upper=3.1416 effort=30.0 velocity=0.2; type revolute -> fixed
- joint bh_j22_joint: limit lower=0.0 upper=2.44 effort=30.0 velocity=2.0 -> lower=0.0 upper=2.44 effort=30.0 velocity=0.2
- joint bh_j23_joint: limit lower=0.0 upper=0.84 effort=30.0 velocity=2.0 -> lower=0.0 upper=0.84 effort=30.0 velocity=0.2
- joint bh_j32_joint: limit lower=0.0 upper=2.44 effort=30.0 velocity=2.0 -> lower=0.0 upper=2.44 effort=30.0 velocity=0.2
- joint bh_j33_joint: limit lower=0.0 upper=0.84 effort=30.0 velocity=2.0 -> lower=0.0 upper=0.84 effort=30.0 velocity=0.2
